Commit message: add content/robots

File: src/curobo/content/assets/robot/abb_irb2600/abb_irb2600_single.urdf (robot description, URDF)
Before this commit: robot mid_robot_dual_cell, 11 links, 10 joints
Joints:
- joint joint_3: limit lower=-3.12159 upper=1.289 effort=0.0 velocity=3.054 -> lower=-1.09626 upper=1.289 effort=0.0 velocity=3.054
